Commit message: fixed coordinate system for sensors in camera. renamed fisheye to color camera

File: realsense2_camera/urdf/_d435.urdf.xacro (robot description, xacro)
@@ -10,7 +10,7 @@
   <!-- The following values are approximate, and the camera node
    publishing TF values with actual calibrated camera extrinsic values -->
-  <xacro:property name="d435_cam_depth_to_left_ir_offset" value="-0.025"/>
-  <xacro:property name="d435_cam_depth_to_right_ir_offset" value="0.025"/>
-  <xacro:property name="d435_cam_depth_to_fisheye_offset" value="0.040"/>
+  <xacro:property name="d435_cam_depth_to_left_ir_offset" value="0.0"/>
+  <xacro:property name="d435_cam_depth_to_right_ir_offset" value="-0.050"/>
+  <xacro:property name="d435_cam_depth_to_color_offset" value="0.015"/>
   <!-- The following values model the aluminum peripherial case for the
     D435 camera, with the camera joint represented by the actual
@@ -23,5 +23,5 @@
     camera tripod mount -->
   <xacro:property name="d435_cam_depth_px" value="${d435_cam_mount_from_center_offset}"/>
-  <xacro:property name="d435_cam_depth_py" value="-0.0075"/>
+  <xacro:property name="d435_cam_depth_py" value="0.0175"/>
   <xacro:property name="d435_cam_depth_pz" value="${d435_cam_height/2}"/>
   <material name="aluminum">
@@ -97,17 +97,17 @@
     </joint>
     <link name="camera_right_ir_optical_frame"/>
-    <!-- camera fisheye joints and links -->
-    <joint name="camera_fisheye_joint" type="fixed">
-      <origin xyz="0 ${d435_cam_depth_to_fisheye_offset} 0" rpy="0 0 0" />
+    <!-- camera color joints and links -->
+    <joint name="camera_color_joint" type="fixed">
+      <origin xyz="0 ${d435_cam_depth_to_color_offset} 0" rpy="0 0 0" />
       <parent link="camera_depth_frame" />
-      <child link="camera_fisheye_frame" />
+      <child link="camera_color_frame" />
     </joint>
-    <link name="camera_fisheye_frame"/>
-    <joint name="camera_fisheye_optical_joint" type="fixed">
+    <link name="camera_color_frame"/>
+    <joint name="camera_color_optical_joint" type="fixed">
       <origin xyz="0 0 0" rpy="${-M_PI/2} 0 ${-M_PI/2}" />
-      <parent link="camera_fisheye_frame" />
-      <child link="camera_fisheye_optical_frame" />
+      <parent link="camera_color_frame" />
+      <child link="camera_color_optical_frame" />
     </joint>
-    <link name="camera_fisheye_optical_frame"/>
+    <link name="camera_color_optical_frame"/>
   </xacro:macro>
 </robot>

Commit message: Fixed different transforms between xacro and driver

File: realsense2_camera/urdf/_d435.urdf.xacro (robot description, xacro)
@@ -37,5 +37,5 @@
     <link name="camera_link">
       <visual>
-      <origin xyz="${d435_cam_mount_from_center_offset} 0.0 ${d435_cam_height/2}" rpy="${M_PI/2} 0 ${M_PI/2}"/>
+      <origin xyz="0.0 ${-1.0 * d435_cam_depth_py} 0.0" rpy="${M_PI/2} 0 ${M_PI/2}"/>
         <geometry>
           <!-- <box size="${d435_cam_width} ${d435_cam_height} ${d435_cam_depth}"/> -->
@@ -46,5 +46,5 @@
       </visual>
       <collision>
-        <origin xyz="0.0 0.0 ${d435_cam_height/2}" rpy="0 0 0"/>
+        <origin xyz="${-1.0 * d435_cam_depth_px} ${-1.0 * d435_cam_depth_py} 0.0" rpy="0 0 0"/>
         <geometry>
         <box size="${d435_cam_depth} ${d435_cam_width} ${d435_cam_height}"/>
@@ -60,5 +60,5 @@
     <!-- camera depth joints and links -->
     <joint name="camera_depth_joint" type="fixed">
-      <origin xyz="${d435_cam_depth_px} ${d435_cam_depth_py} ${d435_cam_depth_pz}" rpy="0 0 0"/>
+      <origin xyz="0 0 0" rpy="0 0 0"/>
       <parent link="camera_link"/>
       <child link="camera_depth_frame" />

Commit message: add bottom_screw joint to _d435.urdf.xacro

File: realsense2_camera/urdf/_d435.urdf.xacro (robot description, xacro)
@@ -33,9 +33,15 @@
       <xacro:insert_block name="origin" />
       <parent link="${parent}"/>
+      <child link="camera_bottom_screw_frame" />
+    </joint>
+    <link name="camera_bottom_screw_frame"/>
+    <joint name="camera_link_joint" type="fixed">
+      <origin xyz="0 ${d435_cam_depth_py} ${d435_cam_depth_pz}" rpy="0 0 0"/>
+      <parent link="camera_bottom_screw_frame"/>
       <child link="camera_link" />
     </joint>
     <link name="camera_link">
       <visual>
-      <origin xyz="0.0 ${-1.0 * d435_cam_depth_py} 0.0" rpy="${M_PI/2} 0 ${M_PI/2}"/>
+      <origin xyz="${d435_cam_mount_from_center_offset} ${-d435_cam_depth_py} 0" rpy="${M_PI/2} 0 ${M_PI/2}"/>
         <geometry>
           <!-- <box size="${d435_cam_width} ${d435_cam_height} ${d435_cam_depth}"/> -->

Commit message: Fixed d435 collision position

File: realsense2_camera/urdf/_d435.urdf.xacro (robot description, xacro)
@@ -52,5 +52,5 @@
       </visual>
       <collision>
-        <origin xyz="${-1.0 * d435_cam_depth_px} ${-1.0 * d435_cam_depth_py} 0.0" rpy="0 0 0"/>
+        <origin xyz="0 ${-d435_cam_depth_py} 0" rpy="0 0 0"/>
         <geometry>
         <box size="${d435_cam_depth} ${d435_cam_width} ${d435_cam_height}"/>
