Commit message: correctred .stl filename

File: realsense2_camera/urdf/_d415.urdf.xacro (robot description, xacro)
@@ -40,5 +40,5 @@
         <geometry>
           <!-- <box size="${d415_cam_width} ${d415_cam_height} ${d415_cam_depth}"/> -->
-	         <mesh filename="package://realsense2_camera/meshes/d415_g.stl" />
+	         <mesh filename="package://realsense2_camera/meshes/d415.stl" />
         </geometry>
         <material name="aluminum"/>

Commit message: fix transform between urdf and driver

File: realsense2_camera/urdf/_d415.urdf.xacro (robot description, xacro)
@@ -33,9 +33,15 @@
       <xacro:insert_block name="origin" />
       <parent link="${parent}"/>
+      <child link="camera_bottom_screw_frame" />
+    </joint>
+    <link name="camera_bottom_screw_frame"/>
+    <joint name="camera_link_joint" type="fixed">
+      <origin xyz="0 ${d415_cam_depth_py} ${d415_cam_depth_pz}" rpy="0 0 0"/>
+      <parent link="camera_bottom_screw_frame"/>
       <child link="camera_link" />
     </joint>
     <link name="camera_link">
       <visual>
-      <origin xyz="${d415_cam_mount_from_center_offset} 0.0 ${d415_cam_height/2}" rpy="${M_PI/2} 0 ${M_PI/2}"/>
+      <origin xyz="${d415_cam_mount_from_center_offset} ${-d415_cam_depth_py} 0" rpy="${M_PI/2} 0 ${M_PI/2}"/>
         <geometry>
           <!-- <box size="${d415_cam_width} ${d415_cam_height} ${d415_cam_depth}"/> -->
@@ -45,5 +51,5 @@
       </visual>
       <collision>
-        <origin xyz="0.0 0.0 ${d415_cam_height/2}" rpy="0 0 0"/>
+        <origin xyz="0 ${-d415_cam_depth_py} 0" rpy="0 0 0"/>
         <geometry>
         <box size="${d415_cam_depth} ${d415_cam_width} ${d415_cam_height}"/>
@@ -59,5 +65,5 @@
     <!-- camera depth joints and links -->
     <joint name="camera_depth_joint" type="fixed">
-      <origin xyz="${d415_cam_depth_px} ${d415_cam_depth_py} ${d415_cam_depth_pz}" rpy="0 0 0"/>
+      <origin xyz="0 0 0" rpy="0 0 0"/>
       <parent link="camera_link"/>
       <child link="camera_depth_frame" />
